Commit message: Add preview functionality for inverse kinematics and update URDF joint definitions

File: src/assets/robotarm_corrected.urdf (robot description, URDF)
Before this commit: robot robotarm, 6 links, 5 joints
Joints:
- removed joint joint_1
- removed joint joint_2
- removed joint joint_3
- removed joint joint_4
- added joint EL1: type revolute, parent link_3, child link_4, origin xyz=0 0 -2.8 rpy=0 0 0, axis 0 1 0, limit lower=-3.15 upper=3.15 effort=0.5 velocity=1.0
- added joint SH1: type revolute, parent base_link, child link_1, origin xyz=0 0 0 rpy=0 0 0, axis 0 1 0, limit lower=-3.15 upper=3.15 effort=0.5 velocity=1.0
- added joint SH2: type revolute, parent link_1, child link_2, origin xyz=0 1 0 rpy=0 0 0, axis 1 0 0, limit lower=-3.15 upper=3.15 effort=0.5 velocity=1.0
- added joint SH3: type revolute, parent link_2, child link_3, origin xyz=1.15 0 0.3 rpy=0 0 0, axis 0 0 1, limit lower=-3.15 upper=3.15 effort=0.5 velocity=1.0
